File: board/cat_tracker_board.kicad_pcb (KiCad board)
At the start: 2 copper layers, 0 parts

Commit message: First pass at a through-hole board layout.
Parts:
- added 10K1: R, Resistors_ThroughHole:Resistor_Horizontal_RM10mm, F.Cu at (154.9, 109.2)
- added C1: 0.1u, Capacitors_ThroughHole:C_Disc_D12_P7.75, F.Cu at (162.6, 128.3)
- added CON1: AVR-ISP-6, Pin_Headers:Pin_Header_Straight_2x03, F.Cu at (160.0, 104.1)
- added IC1: ATMEGA328-P, Housings_DIP:DIP-28_W7.62mm_LongPads, F.Cu at (167.6, 100.3)
- added P1: GPS_NMEA, Pin_Headers:Pin_Header_Straight_1x04, F.Cu at (154.9, 123.2)
- added P2: MicroSD Card Adapter, Pin_Headers:Pin_Header_Straight_1x06, F.Cu at (158.8, 139.7)
- added P4: BATTERY, Pin_Headers:Pin_Header_Straight_1x02, F.Cu at (160.0, 99.1)
- added SW1: RESET, Buttons_Switches_ThroughHole:SW_PUSH_SMALL, F.Cu at (158.8, 116.8)
- added X1: 16Mhz XTAL, Crystals:Crystal_HC49-U_Vertical_3Pin, F.Cu at (160.0, 134.6)
